File: PatrolVMU.kicad_pcb (KiCad board)
At the start: 2 copper layers, 0 parts

Commit message: finished preliminarly
Parts:
- added C1: 100nf, Capacitor_SMD:C_0805_2012Metric, F.Cu at (129.4, 110.5)
- added C10: 10pF, Capacitor_SMD:C_0805_2012Metric, F.Cu at (142.2, 123.0)
- added C11: 0.1uF, Capacitor_SMD:C_0805_2012Metric, F.Cu at (133.2, 114.5)
- added C12: 0.001uF, Capacitor_SMD:C_0805_2012Metric, F.Cu at (127.3, 98.2)
- added C13: 1uF, Capacitor_SMD:C_0805_2012Metric, F.Cu at (131.5, 94.7)
- added C2: 10nf, Capacitor_SMD:C_0805_2012Metric, F.Cu at (145.1, 129.4)
- added C3: 100nf, Capacitor_SMD:C_0805_2012Metric, F.Cu at (132.2, 132.2)
- added C7: 10uf, Capacitor_SMD:C_0805_2012Metric, F.Cu at (122.7, 100.9)
- added C8: 0.1uF, Capacitor_SMD:C_0805_2012Metric, F.Cu at (122.7, 97.4)
- added C9: 10pF, Capacitor_SMD:C_0805_2012Metric, F.Cu at (133.5, 123.0)
- added D1: SMBJ26A, Diode_SMD:D_SMB, F.Cu at (130.9, 107.1)
- added D2: SMBJ26A, Diode_SMD:D_SMB, F.Cu at (137.9, 132.3)
- added D4: Red, LED_SMD:LED_0805_2012Metric, F.Cu at (125.0, 97.4)
- added J1: C-OBD-II-16M, C-OBD-II-16M:COMTECH_C-OBD-II-16M, F.Cu at (139.1, 84.5)
- added J2: Conn_01x03_Pin, Jumper:SolderJumper-3_P1.3mm_Bridged2Bar12_Pad1.0x1.5mm, F.Cu at (138.2, 110.8)
- added Q1: BC549CTA, BC549CTA:BC33740TA, F.Cu at (139.4, 95.7)
- added Q2: BC549CTA, BC549CTA:BC33740TA, F.Cu at (141.8, 104.4)
- added R1: 6k8, Capacitor_SMD:C_0805_2012Metric, F.Cu at (127.3, 94.7)
- added R10: 1k, Capacitor_SMD:C_0805_2012Metric, F.Cu at (142.3, 110.5)
- added R11: 4k7, Capacitor_SMD:C_0805_2012Metric, F.Cu at (142.3, 108.4)
- added R12: 1k, Capacitor_SMD:C_0805_2012Metric, F.Cu at (138.8, 108.4)
- added R13: 10k, Capacitor_SMD:C_0805_2012Metric, F.Cu at (129.4, 94.7)
- added R14: 4k7, Capacitor_SMD:C_0805_2012Metric, F.Cu at (129.4, 98.2)
- added R15: 10k, Capacitor_SMD:C_0805_2012Metric, F.Cu at (129.4, 121.5)
- added R16: 10k, Capacitor_SMD:C_0805_2012Metric, F.Cu at (129.4, 123.6)
- added R17: 10k, Capacitor_SMD:C_0805_2012Metric, F.Cu at (129.4, 125.7)
- added R18: 100, Resistor_SMD:R_2512_6332Metric, F.Cu at (131.0, 102.8)
- added R19: 10k, Capacitor_SMD:C_0805_2012Metric, F.Cu at (145.1, 125.8)
- added R2: 4k7, Capacitor_SMD:C_0805_2012Metric, F.Cu at (131.5, 98.2)
- added R20: 200k, Capacitor_SMD:C_0805_2012Metric, F.Cu at (145.1, 132.9)
- added R21: 33k, Capacitor_SMD:C_0805_2012Metric, F.Cu at (142.8, 131.8)
- added R22: 1M, Capacitor_SMD:C_0805_2012Metric, F.Cu at (123.8, 132.1)
- added R23: 180k, Capacitor_SMD:C_0805_2012Metric, F.Cu at (126.1, 130.1)
- added R24: 180k, Capacitor_SMD:C_0805_2012Metric, F.Cu at (126.1, 133.7)
- added R3: 1k, Capacitor_SMD:C_0805_2012Metric, F.Cu at (143.5, 92.3)
- added R4: 4k7, Capacitor_SMD:C_0805_2012Metric, F.Cu at (143.5, 96.0)
- added R5: 1k, Capacitor_SMD:C_0805_2012Metric, F.Cu at (143.5, 99.7)
- added R6: 1k, Capacitor_SMD:C_0805_2012Metric, F.Cu at (123.4, 94.4)
- added R7: 10k, Capacitor_SMD:C_0805_2012Metric, F.Cu at (129.4, 127.8)
- added R8: 10M, Capacitor_SMD:C_0805_2012Metric, F.Cu at (137.9, 123.0)
- added R9: 10k, Capacitor_SMD:C_0805_2012Metric, F.Cu at (129.4, 119.4)
- added U1: ESP32-C3, Waveshare-ESP32:Waveshare-ESP32-C3-Zero, F.Cu at (115.3, 116.5)
- added U2: CD4060BNSR, CD4060BNSR:SOIC127P780X200-16N, F.Cu at (139.9, 117.0)
- added U3: L7805, Package_TO_SOT_SMD:TO-263-2, F.Cu at (111.2, 96.9)
- added U4: LM358ST, LM358ST:SOP65P490X110-8N, F.Cu at (134.5, 96.5)
- added U5: INA226, Package_SO:VSSOP-10_3x3mm_P0.5mm, F.Cu at (129.4, 114.8)
- added U6: TLV7031DBV, Package_TO_SOT_SMD:SOT-23-5, F.Cu at (129.2, 132.1)
- added Y1: 2.4576M, Crystal:Crystal_HC49-4H_Vertical, F.Cu at (135.2, 127.0)
Routing:
- net GND: track 0.00 -> 200.2 mm, vias 0 -> 2
- net +5V: track 0.00 -> 91.4 mm, vias 0 -> 4
- net OBD_ignition: track 0.00 -> 75.5 mm, vias 0 -> 2
- net ESP_Tx: track 0.00 -> 51.5 mm, vias 0 -> 2
- net OBD_12v: track 0.00 -> 50.5 mm, vias 0 -> 2
- net OBD_clock: track 0.00 -> 49.9 mm, vias 0 -> 1
- net OBD_rx: track 0.00 -> 38.9 mm
- net ESP_Rx: track 0.00 -> 37.9 mm, vias 0 -> 2
- net ESP_I2C_SCL: track 0.00 -> 33.6 mm, vias 0 -> 2
- net ESP_I2C_SDA: track 0.00 -> 31.8 mm
- net +3.3V: track 0.00 -> 28.5 mm
- net OBD_IGN_SIG: track 0.00 -> 21.7 mm
- net OBD_tx: track 0.00 -> 21.3 mm, vias 0 -> 2
- net Net-(U2-~{O}): track 0.00 -> 19.4 mm
- net Net-(U5-A1): track 0.00 -> 17.8 mm, vias 0 -> 2
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